File: Hardware/0. Project/NoteIt.sch (EAGLE design)
At the start: 85 parts, among them CN2 MicroSD Card, CN3 MicroSD Card, IC1 MSP430FR4133IG48R, IC2 MCP73831/2, IC5 S-8261ACMMD-G4MT2U, J2 USB4110-GF-A_REVB, Q1 ABS07-120-32.768KHZ-T, Q2 SI2374DS, Q3 SI2374DS, Q4 BC817, SW1 KY-040, U1 TP4056, U2 MSP430G2553, U3 DW01A-G, U4 FS8205A, U5 TLV75530PDBVR, U6 GL823, U7 RT9193-33GB, U8 ADG774, U9 ADG774, X3 microUSB

Commit message: Migrating MCU to FR2476
Parts:
- removed IC1: MSP430FR4133IG48R, MSP430FR4133:MSP430FR4133
- removed Q1: ABS07-120-32.768KHZ-T, crystal-geyer_V1_0:KX-327-NHF
- added C21, C22: 10uF x 10V, My-RLC:C_0603
- added C23: 1nF x 50V, My-RLC:C_0603
- added CN5, CN7: 1x4, pinhead:PINHD-1X4
- added R19: 47k (5%), My-RLC:R_0603
- added TP7, TP8: TPB1,27, testpad:TPB1,27
- added U10: MSP430FR2476TPTR, MSP430FR2476TPTR:MSP430FR2476TPTR
- C5, C6: value C0805C220K5HACTU -> 100nF x 50V; device rcl:C-EUC0805 -> My-RLC:C_0603; PN (none) -> C0603C104M5RACTU
Connections:
- new net ADC_CURRENT_L1: U10.P5.3/UCB1CLK/TA3.0/A10
- new net ADC_CURRENT_L2: U10.P4.3/UCB1SOMI/UCB1SCL/TB0.5/A8
- new net ADC_CURRENT_L3: U10.P1.6/UCA0CLK/TA1CLK/TDI/TCLK/A6
- new net ADC_VOLTAGE_L1: U10.P5.4/UCB1STE/TA3CLK/A11
- new net ADC_VOLTAGE_L2: U10.P4.4/UCB1SIMO/UCB1SDA/TB0.6/A9
- new net ADC_VOLTAGE_L3: U10.P1.7/UCA0STE/SMCLK/TDO/A7
- new net ADC_VREF: C22.1, C6.1, U10.P1.0/UCB0STE/TA0CLK/A0/VEREF+
- new net BUTTON_METER_CALIBRATION: U10.P1.2/UCB0SIMO/UCB0SDA/TA0.2/A2/VEREF-
- new net CMP_ZERO_CROSSING_L1: U10.P6.0/TA2.2/COMP0.3
- new net CMP_ZERO_CROSSING_L2: U10.P5.7/TA2.1/COMP0.2
- new net CMP_ZERO_CROSSING_L3: U10.P2.2/ACLK/COMP0.1
- new net GPIO_MSP430_EXTERNAL_USE: U10.P3.0/TA2.2
- new net LED_GREEN: U10.P5.0/UCA0CLK/TB0.2
- new net LED_RED: U10.P5.6/UCB0STE/TA2.0
- new net MSP<->ESP32_UART_RX: U10.P5.1/UCA0RXD/UCA0SOMI/TB0.3
- new net MSP<->ESP32_UART_TX: U10.P5.2/UCA0TXD/UCA0SIMO/TB0.4
- new net N$15: TP7.TP, U10.P1.4/UCA0TXD/UCA0SIMO/TA1.2/TCK/A4/VREF+
- new net N$34: TP8.TP, U10.P1.5/UCA0RXD/UCA0SOMI/TA1.1/TMS/A5
- new net RELAY_CUT_OFF: U10.P3.3/TA2.1
- new net SBWTDIO: C23.1, CN7.3, R19.2, U10.!RST!/NMI/SBWTDIO
- new net UART_RX_MSP430_EXTERNAL_USE: CN5.2, U10.P2.5/UCA1RXD/UCA1SOMI
- new net UART_TX_MSP430_EXTERNAL_USE: CN5.3, U10.P2.6/UCA1TXD/UCA1SIMO
- net +5V: now also CN5.1
- net 0V: now also C21.2, C22.2, C23.2, C5.2, C6.2, CN5.4, CN7.1, U10.DVSS
- net 3.3V: now also C21.1, C5.1, CN7.4, R19.1, U10.DVCC
- net 3V: no longer IC1.DVCC
- net GND: no longer C5.2, C6.2, IC1.DVSS
- net MCU_RESET: no longer IC1.RST/NMI/SBWTDIO
- net SBWTCK: now also CN7.2, U10.TEST/SBWTCK; no longer IC1.TEST/SBWTCK
- net XIN: now also U10.P2.1/XIN; no longer C6.1, IC1.P4.2/XOUT, Q1.1
- net XOUT: now also U10.P2.0/XOUT; no longer C5.1, IC1.P4.1/XIN, Q1.2
Other:
- note removed: "22pF"
- note removed: "32.768 kHz"
- moved on the sheet: C5, C6

Commit message: Signals names added to MCU (matching with firmware)
Parts:
- removed BT1: 3.7V x 850mAh, Battery-Cable:BATTERY-3PIN
- removed C13: 10UF, rcl:C-EUC0603
- removed C14: 1uF, rcl:C-EUC0805
- removed C17: 22nF, rcl:C-EUC0805
- removed C18: 1000uF x 10V, rcl:CPOL-EUE2-5
- removed C22: 10uF x 10V, My-RLC:C_0603
- removed C3, C30, C7: 100nF, rcl:C-EUC0603
- removed C4: C0805C102J5GAC7210, rcl:C-EUC0805
- removed CN1: (no value), pinhead:PINHD-1X4
- removed CN5: 1x4, pinhead:PINHD-1X4
- removed J1: (no value), con-jack:JACK-PLUG0
- removed J2: USB4110-GF-A_REVB, USB-C:USB4110-GF-A_REVB
- removed R1: 10k (5%), rcl:R-EU_R0603
- removed R10: 100R, rcl:R-EU_R0603
- removed R18: 100k, rcl:R-EU_R0603
- removed R2: CR0805-JW-473ELF, rcl:R-EU_R0805
- removed R3: 1k2 (5%), rcl:R-EU_R0603
- removed R4: 1k (5%), rcl:R-EU_R0603
- removed R5: 5k, resistor:R-TRIMM64P
- removed R7: 10k, ptc-ntc:NTC640
- removed R9: 1k, rcl:R-EU_R0603
- removed TP7, TP8: TPB1,27, testpad:TPB1,27
- removed U$1: DISPLAY-OLED-128X64, diy-modules:DISPLAY-OLED-128X64
- removed U1: TP4056, TP4056:TP4056
- removed U2: MSP430G2553, SamacSys_Parts:MSP430G2553IN20
- removed U3: DW01A-G, DW01A-G:DW01A-G
- removed U4: FS8205A, FS8205A:FS8205A
- removed U7: RT9193-33GB, RT9193-33GB:RT9193-33GB
- added C25: 100nF, rcl:C-EUC0603
- added DS1: SSD1306, diy-modules:DISPLAY-OLED-128X64
- added X2: 32.768 kHz, crystal-geyer_V1_0:CRYSTAL-MINI
- C2: value 100nF -> 22pF x 100V; device rcl:C-EUC0603 -> My-RLC:C_0603; PN (none) -> C0603C220J1GACTU
- C6: value 100nF x 50V -> 22pF x 100V; PN C0603C104M5RACTU -> C0603C220J1GACTU
Connections:
- net ADC_CURRENT_L1 renamed SPI_DISPLAY_CLK
- net ADC_CURRENT_L2 renamed SPI_DISPLAY_SOMI
- net ADC_CURRENT_L3 renamed SPI_SDCARD_CLK
- net ADC_VOLTAGE_L1 renamed !SPI_DISPLAY_CS
- net ADC_VOLTAGE_L2 renamed SPI_DISPLAY_SIMO
- net ADC_VOLTAGE_L3 renamed !SPI_SDCARD_CS
- net BUTTON_METER_CALIBRATION renamed I2C_RTC_SDA
- removed net !BAT_CHARGING!: U1.!CHRG
- removed net !BAT_STANDBY!: U1.!STDBY
- removed net 3V: CN1.1, R2.1
- removed net ADC_VREF: C22.1, C6.1, U10.P1.0/UCB0STE/TA0CLK/A0/VEREF+
- removed net BATTERY_ADC_VOLTAGE: U2.P1.0
- removed net BAT_OVER_CHARGE_DETECTED: U3.OC, U4.G2
- removed net BAT_OVER_DISCHARGE_DETECTED: U3.OD, U4.G1
- removed net CMP_ZERO_CROSSING_L1: U10.P6.0/TA2.2/COMP0.3
- removed net CMP_ZERO_CROSSING_L2: U10.P5.7/TA2.1/COMP0.2
- removed net CMP_ZERO_CROSSING_L3: U10.P2.2/ACLK/COMP0.1
- removed net EXTERNAL_DEVICE_UART_TX: U2.P1.1
- removed net GND: C13.2, C14.2, C17.2, C18.-, C2.2, C4.2, CN1.4, J1.1, J1.2, R18.1, R3.1, R5.A, R5.S, R7.1, R9.1, U1.GND, U4.S2_1, U7.GND
- removed net GPIO_MSP430_EXTERNAL_USE: U10.P3.0/TA2.2
- removed net GPIO_ROTARY_ENCODER_SIGNAL-A: SW1.A, U2.P2.1
- removed net GPIO_ROTARY_ENCODER_SIGNAL-B: SW1.B, U2.P2.2
- removed net GPIO_ROTARY_ENCODER_SWITCH: SW1.SW1, U2.P2.0
- removed net LED_GREEN: U10.P5.0/UCA0CLK/TB0.2
- removed net LED_RED: U10.P5.6/UCB0STE/TA2.0
- removed net MCU_RESET: C4.1, CN1.2, R2.2
- removed net MSP<->ESP32_UART_RX: U10.P5.1/UCA0RXD/UCA0SOMI/TB0.3
- removed net MSP<->ESP32_UART_TX: U10.P5.2/UCA0TXD/UCA0SIMO/TB0.4
- removed net N$15: TP7.TP, U10.P1.4/UCA0TXD/UCA0SIMO/TA1.2/TCK/A4/VREF+
- removed net N$16: R4.1, R5.E, R7.2, U1.TEMP1
- removed net N$2: U2.P1.2
- removed net N$34: TP8.TP, U10.P1.5/UCA0RXD/UCA0SOMI/TA1.1/TMS/A5
- removed net N$7: R9.2, U3.CS
- removed net N$8: C7.1, R10.2, U3.VCC
- removed net RELAY_CUT_OFF: U10.P3.3/TA2.1
- removed net SBWTCK: CN1.3, CN7.2, U10.TEST/SBWTCK
- removed net SBWTDIO: C23.1, CN7.3, R19.2, U10.!RST!/NMI/SBWTDIO
- removed net UART_RX_MSP430_EXTERNAL_USE: CN5.2, U10.P2.5/UCA1RXD/UCA1SOMI
- removed net UART_TX_MSP430_EXTERNAL_USE: CN5.3, U10.P2.6/UCA1TXD/UCA1SIMO
- removed net V_BAT+: BT1.+, C13.1, C14.1, R10.1, R18.2, U1.BAT, U7.EN, U7.VIN
- removed net V_BAT-: BT1.-, C7.2, U3.GND, U4.S1_1
- removed net V_EXTERNAL_SUPPLY: C2.1, J1.3, R4.2, U1.CE, U1.VCC
- removed net XIN: U10.P2.1/XIN
- removed net XOUT: U10.P2.0/XOUT
- new net !GPIO_OLED_RESET: DS1.!RST, U10.P6.2/TB0.0
- new net ADC_BATTERY_VOLTAGE: U10.P1.0/UCB0STE/TA0CLK/A0/VEREF+
- new net GPIO_EXTERNAL_SUPPLY_DETECT: U10.P4.7/UCA0STE/TB0.1
- new net GPIO_OLED_TRANSMISSION_MODE: DS1.DC, U10.P3.7/TA3.2
- new net GPIO_ROTARY_ENCODER_BUTTON: SW1.SW1, U10.P4.0/TA3.1
- new net GPIO_ROTARY_ENCODER_SIGNAL_A: SW1.A, U10.P4.1/TA3.0
- new net GPIO_ROTARY_ENCODER_SIGNAL_B: SW1.B, U10.P4.2/TA3CLK
- new net GPIO_SDCARD_DETECT: U10.P4.6/UCB0SIMO/UCB0SDA/TA3.1
- new net GPIO_USB_DETECT: U10.P4.5/UCB0SOMI/UCB0SCL/TA3.2
- new net I2C_RTC_SCL: U10.P1.3/UCB0SOMI/UCB0SCL/MCLK/A3
- new net OLED_SPI_MOSI: DS1.MOSI
- new net OLED_SPI_SCLK: DS1.SCLK
- new net SPI_SDCARD_SIMO: U10.P1.4/UCA0TXD/UCA0SIMO/TA1.2/TCK/A4/VREF+
- new net SPI_SDCARD_SOMI: U10.P1.5/UCA0RXD/UCA0SOMI/TA1.1/TMS/A5
- new net UART_DATALOGGER_RX: U10.P2.5/UCA1RXD/UCA1SOMI
- new net XTAL_IN: C2.1, U10.P2.1/XIN, X2.1
- new net XTAL_OUT: C6.1, U10.P2.0/XOUT, X2.2
- net !SDCARD_CARD_DETECT!: no longer U2.P2.3
- net +5V: no longer CN5.1
- net 0V: now also C2.2, C25.2, DS1.GND; no longer C22.2, C3.1, C41.2, C42.2, CN5.4, LED4.C, U2.DVSS, X3.GND
- net 3.3V: now also C25.1, DS1.VCC; no longer C18.+, C3.2, U2.DVCC, U7.VOUT
- net 5V: no longer C41.1, C42.1, R25.2, X3.VBUS
- net ICSP_SBWTCK: now also CN7.2, U10.TEST/SBWTCK; no longer U2.TEST/SBWTCK
- net ICSP_SBWTDIO: now also C23.1, CN7.3, R19.2, U10.!RST!/NMI/SBWTDIO; no longer U2.!RST!/NMI/SBWTDIO
- net N$4: now also C41.1, C42.1, R25.2, X3.VBUS; no longer C17.1, U7.BP
- net N$6: now also C41.2, C42.2, LED4.C, X3.GND; no longer R3.2, U1.PROG2
- net OLED_SPI_!CS!: now also DS1.!CS; no longer U2.P2.4
- net SDCARD_SPI_!CS!: no longer U2.P2.5
- net SDCARD_SPI_MISO: no longer U2.P1.6
- net SDCARD_SPI_MOSI: no longer U2.P1.7
- net SDCARD_SPI_SCLK: no longer U2.P1.5
Other:
- note added: "TODO: Level shifter at RXD?"
- note removed: ""SIMO""
- note removed: ""SOMI""
- note removed: "*"
- note removed: "1 nF"
- note removed: "47k"
- note removed: "BATTERY CHARGER"
- note removed: "BATTERY PROTECTION"
- note removed: "From TP4056 Datasheet"
- note removed: "IN-CIRCUIT SERIAL PROGRAMMING"
- note removed: "If TEMP pin’s voltage is below 45% or above 80% of supply voltage VCC for more than 0.15S, this means that battery’s temperature is too high or too low, charging is suspended."
- note removed: "RECHARGEABLE BATTERY"
- note removed: "TODO: Change to SPI model"
- note removed: "TODO: Level shifter at TXD"
- note removed: "VOLTAGE REGULATOR"
- moved on the sheet: C1, C19, C2, C21, C23, C24, C39, C41, C42, C5, C6, C9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

Commit message: WIP
Other:
- moved on the sheet: C2, C25, C6, CN7, DS1, SW1, U8, U9, X2

Commit message: USB/MCU <--> Micro-SD Card Interface added
Parts:
- removed C1, C20, C28, C31, C42: 100nF, rcl:C-EUC0603
- removed C41: 10uF, rcl:C-EUC0603
- removed CN2, CN3: MicroSD Card, Micro SD:MICROSD-PUSH-OUT
- removed LED4: (no value), led:LEDSML0603
- removed R21, R6, R8: 10k (5%), rcl:R-EU_R0603
- removed R23: 100k (5%), rcl:R-EU_R0603
- removed R25: 1k, rcl:R-EU_R0603
- removed R28, R29: 22R, rcl:R-EU_R0603
- removed U8, U9: ADG774, ADG774:ADG774
- removed X3: microUSB, microbuilder:USB_MICRO_20329_V2
- added C3, C4: 100nF, rcl:C-EUC0603
- added CN1: Micro-SD Card, Micro SD:MICROSD-PUSH-OUT
- added U4: TS3A27518EPWR, TS3A27518EPWR:TS3A27518EPWR
Connections:
- removed net !SDCARD_SPI_CS!: U8.S4B
- removed net !SPI_SDCARD_CS: U10.P1.7/UCA0STE/SMCLK/TDO/A7
- removed net +5V: C1.1, C20.1, C28.1, C31.1, CN2.4, CN3.4, R11.2, R21.2, R6.2, R8.2, U8.VDD, U9.VDD
- removed net 5V: IC2.VDD, R33.2
- removed net MUX_MCU2USB: Q4.C, R11.1, U8.IN, U9.IN
- removed net N$21: LED4.A, R25.1
- removed net N$22: R28.2, X3.D+
- removed net N$23: R29.2, X3.D-
- removed net N$4: C41.1, C42.1, R25.2, X3.VBUS
- removed net N$6: C41.2, C42.2, LED4.C, X3.GND
- removed net SDCARD_CLK: CN3.5, U9.D2
- removed net SDCARD_CMD/MOSI: CN3.3, R21.1, U9.D1
- removed net SDCARD_DAT0/MISO: CN3.7, R6.1, U8.D1
- removed net SDCARD_DAT1: CN3.8, U8.D2
- removed net SDCARD_DAT2: CN3.1, U8.D3
- removed net SDCARD_DAT3/!CS!: CN3.2, U8.D4
- removed net SDCARD_SPI_!CS!: CN2.2
- removed net SDCARD_SPI_CLK: U9.S2B
- removed net SDCARD_SPI_MISO: CN2.7, R23.1, U8.S1B
- removed net SDCARD_SPI_MOSI: CN2.3, U9.S1B
- removed net SDCARD_SPI_SCLK: CN2.5
- removed net SPI_SDCARD_CLK: U10.P1.6/UCA0CLK/TA1CLK/TDI/TCLK/A6
- removed net SPI_SDCARD_SIMO: U10.P1.4/UCA0TXD/UCA0SIMO/TA1.2/TCK/A4/VREF+
- removed net SPI_SDCARD_SOMI: U10.P1.5/UCA0RXD/UCA0SOMI/TA1.1/TMS/A5
- removed net USB_D+: R28.1
- removed net USB_D-: R29.1
- removed net USB_VDD: C16.2, R14.2, R15.1, U6.VBUS, X1.1
- new net !CONNECT_SDCARD_TO_USB: Q4.C, R11.1, U4.1N1, U4.1N2
- new net MCU_!SPI_SDCARD_CS: U10.P1.7/UCA0STE/SMCLK/TDO/A7, U4.NO6
- new net MCU_SPI_SDCARD_SCLK: U10.P1.6/UCA0CLK/TA1CLK/TDI/TCLK/A6, U4.NO1
- new net MCU_SPI_SDCARD_SIMO: U10.P1.4/UCA0TXD/UCA0SIMO/TA1.2/TCK/A4/VREF+, U4.NO2
- new net MCU_SPI_SDCARD_SOMI: U10.P1.5/UCA0RXD/UCA0SOMI/TA1.1/TMS/A5, U4.NO3
- new net N$15: CN1.CMD, U4.COM2
- new net N$16: CN1.DAT0, U4.COM3
- new net N$2: CN1.CLK, U4.COM1
- new net N$20: CN1.DAT1, U4.COM4
- new net N$7: CN1.DAT2, U4.COM5
- new net N$8: CN1.DAT3, U4.COM6
- new net VUSB: C16.2, IC2.VDD, R14.2, R15.1, R33.2, U6.VBUS, X1.1
- net !SDCARD_CARD_DETECT!: now also CN1.9; no longer CN2.9, CN3.9, R8.1
- net 0V: now also C3.1, C4.1, CN1.CHASSI, CN1.GND, U4.!EN, U4.GND; no longer C1.2, C20.2, C28.2, C31.2, CN2.10, CN2.6, CN3.10, CN3.6, R23.2, U8.!EN!, U8.VSS, U9.!EN!, U9.VSS
- net 3.3V: now also C3.2, C4.2, CN1.VDD, R11.2, U4.VCC
- net USB_CLK: now also U4.NC1; no longer U9.S2A
- net USB_CMD: now also U4.NC2; no longer U9.S1A
- net USB_DAT0: now also U4.NC3; no longer U8.S1A
- net USB_DAT1: now also U4.NC4; no longer U8.S2A
- net USB_DAT2: now also U4.NC5; no longer U8.S3A
- net USB_DAT3: now also U4.NC6; no longer U8.S4A
Other:
- note added: "AUTOMATIC INTERFACES SWITCH"
- note added: "MCU INTERFACE"
- note added: "USB INTERFACE"
- note removed: "Micro SD-Card interface"
- note removed: "Micro SD-Card to USB Interface"
- note removed: "[MCU or USB] <--> [Micro SD-Card] Communication (MCU as default)"
- moved on the sheet: C10, C11, C12, C15, C16, L1, LED2, Q4, R11, R14, R15, R16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

Commit message: USB C added + UART Rx (datalogger input) level shifter added
Parts:
- removed X1: (no value), con-berg:PN87520
- added C1: 4.7nF, rcl:C-EUC0603
- added CN2: (no value), con-ptr500:AK500/2-H
- added CN3: USB 3.2 Gen 2 Type C Receptacle, USB C CONNECOTR:USB4080-03-A
- added R1, R2: 5k1 (5%), rcl:R-EU_R0603
- added R3: 1M, rcl:R-EU_R0603
- added U1: SN74AHC1G125DRLR, SN74AHC1G125DRLR:SN74AHC1G125
Connections:
- removed net N$11: U6.USB_P, X1.3
- new net N$21: CN3.CC2, R2.1
- new net N$4: CN2-1.KL, U1.A
- new net N$6: CN3.CC1, R1.1
- new net USB_N: CN3.DN1, CN3.DN2, U6.USB_N
- new net USB_P: CN3.DP1, CN3.DP2, U6.USB_P
- net 0V: now also C1.1, CN2-2.KL, CN3.GND_A, CN3.GND_B, R1.2, R2.2, R3.2, U1.!OE, U1.GND; no longer X1.4
- net 3.3V: now also U1.VDD
- net N$10: now also C1.2, CN3.SHIELD, R3.1; no longer U6.USB_N, X1.2
- net UART_DATALOGGER_RX: now also U1.Y
- net VUSB: now also CN3.VBUS_A, CN3.VBUS_B; no longer X1.1
Other:
- note added: "5V TOLERANT"
- note added: "IQ = 10μA"
- note removed: "TODO: Level shifter at RXD?"
- moved on the sheet: BT2, C10, C11, C12, C15, C16, C19, C24, C3, C39, C4, C8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

Commit message: SD-Card to USB IC (GL823K) package updated
Parts:
- removed C12: 100nF, rcl:C-EUC0603
- removed C23: 1nF x 50V, My-RLC:C_0603
- removed CN7: 1x4, pinhead:PINHD-1X4
- removed L1: BLM15HB221SN1, inductors:BLM15HB221SN1
- removed LED1: (no value), led:LEDSML0603
- removed R16: 680R (5%), rcl:R-EU_R0603
- removed R19: 47k (5%), My-RLC:R_0603
- removed R33: 470R, rcl:R-EU_R0603
- removed U6: GL823, GL823:GL823(B)HG
- added C13: 1nF x 50V, My-RLC:C_0603
- added C14: 100nF, rcl:C-EUC0805
- added C7: 100nF, rcl:C-EUC0603
- added CN4: ARM 10-pin JTAG Connector, SamacSys_Parts:FTSH-105-01-L-DV-K-TR
- added G1: CR1220, battery:CH291-1220LF
- added R10: 4k7, rcl:R-EU_R0603
- added R18: 10k, rcl:R-EU_R0603
- added R4, R9: 100k, rcl:R-EU_R0603
- added R5: 10k (5%), rcl:R-EU_R0603
- added R6, R7, R8: 47k (5%), My-RLC:R_0603
- added U2: GL823K, SamacSys_Parts:GL823K
- added U8: DS3231/SO, adafruit:DS3231/SO
- C10: value 10uF -> 4.7uF
- C11, C15: value 100nF -> 4.7uF
Connections:
- net !GPIO_OLED_RESET renamed !GPIO_DISPLAY_RESET
- net GPIO_OLED_TRANSMISSION_MODE renamed GPIO_DISPLAY_TRANSMISSION_MODE
- removed net ADC_VBAT: R41.1, R42.2
- removed net GPIO_EXTERNAL_SUPPLY_DETECT: U10.P4.7/UCA0STE/TB0.1
- removed net GPIO_SDCARD_DETECT: U10.P4.6/UCB0SIMO/UCB0SDA/TA3.1
- removed net N$18: R16.1, U6.RREF
- removed net N$19: L1.2, U6.AVDD
- removed net N$24: LED1.A, R33.1
- removed net N$25: IC2.STAT, LED1.C
- removed net N$9 (its old number): C12.2, U6.PMOS
- removed net OLED_SPI_!CS!: DS1.!CS
- removed net OLED_SPI_MOSI: DS1.MOSI
- removed net OLED_SPI_SCLK: DS1.SCLK
- removed net SPI_DISPLAY_CLK: U10.P5.3/UCB1CLK/TA3.0/A10
- removed net SPI_DISPLAY_SOMI: U10.P4.3/UCB1SOMI/UCB1SCL/TB0.5/A8
- new net GPIO_BATTERY_CHARGING_STATUS: IC2.STAT, U10.P4.7/UCA0STE/TB0.1
- new net N$13: C15.2, U2.PMOS
- new net N$22: G1.+, U8.VBAT
- new net SPI_DISPLAY_SCLK: DS1.SCLK, U10.P5.3/UCB1CLK/TA3.0/A10
- net !SDCARD_CARD_DETECT!: now also CN1.!CD, R5.2, U10.P4.6/UCB0SIMO/UCB0SDA/TA3.1; no longer CN1.9, U6.!SD_CD
- net !SPI_DISPLAY_CS: now also DS1.!CS
- net 0V: now also C13.2, C14.1, CN4.3, CN4.5, CN4.7, CN4.9, G1.-, R18.1, R9.1, U2.VSS_1, U2.VSS_2, U8.GND; no longer C10.1, C11.1, C12.1, C23.2, CN7.1, LED2.C, R16.2, U6.GND, U6.GPIO3, U6.GPIO6, U6.SCL, U6.SDA, U6.SD_WP, U6.TEST
- net 3.3V: now also C14.2, CN4.1, R5.1, R6.1, R7.1, R8.1, U8.VDD; no longer CN7.4, R19.1
- net ADC_BATTERY_VOLTAGE: now also R41.1, R42.2
- net GPIO_USB_DETECT: now also R4.1, R9.2
- net I2C_RTC_SCL: now also R8.2, U8.SCL
- net I2C_RTC_SDA: now also R7.2, U8.SDA
- net ICSP_SBWTCK: now also CN4.4; no longer CN7.2
- net ICSP_SBWTDIO: now also C13.1, CN4.6, R6.2; no longer C23.1, CN7.3, R19.2
- net N$12: now also R10.1, R18.2, U2.GPIO; no longer R17.1, U6.LED
- net N$17: now also C10.2, C11.2, R10.2, R17.1, U2.VDD, U2.VDDA; no longer C15.2, U6.!RESET
- net N$5: now also LED2.C, U2.LED; no longer C10.2, C11.2, L1.1, U6.DVDD
- net SPI_DISPLAY_SIMO: now also DS1.MOSI
- net USB_CLK: now also U2.CLK; no longer U6.SD_CLK
- net USB_CMD: now also U2.CMD; no longer U6.SD_CMD
- net USB_DAT0: now also U2.DAT0; no longer U6.SD_D0
- net USB_DAT1: now also U2.DAT1; no longer U6.SD_D1
- net USB_DAT2: now also U2.DAT2; no longer U6.SD_D2
- net USB_DAT3: now also U2.DAT3; no longer U6.SD_D3
- net USB_N: now also U2.DN; no longer U6.USB_N
- net USB_P: now also U2.DP; no longer U6.USB_P
- net VUSB: now also R4.2, U2.5V; no longer R33.2, U6.VBUS
- net XTAL_IN: now also U10.P2.0/XOUT; no longer U10.P2.1/XIN
- net XTAL_OUT: now also U10.P2.1/XIN; no longer U10.P2.0/XOUT
Other:
- note added: "(3V / 37 mAh)"
- note added: "*"
- note added: "- only two pins used; - no overlap between JTAG and I/O pins; - slower than 4-wire JTAG."
- note added: "3.7V ~ 4.2V 230mAh"
- note added: "7-bits Slave Address 0b1101000 0x68"
- note added: "TODO: Add pins to an externsion board with MAX232 connect"
- note added: "Transmission Mode is used to set the display to receive a DATA instruction or a COMMAND instruction from SIMO (MOSI) pin."
- note added: "this is a signal provided by the socket, not the micro-sd card itself."
- note removed: "3.7V ~4.2V 230mAh"
- moved on the sheet: BT2, C1, C10, C11, C15, C16, C19, C2, C21, C24, C25, C3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

Commit message: PCB layout init
Parts:
- C1: value 4.7nF -> (none)
- C10, C11, C15: value 4.7uF -> (none)
- C13: value 1nF x 50V -> (none)
- C14, C16, C19, C25, C3, C39, C4, C7, C8: value 100nF -> (none)
- C2, C6: value 22pF x 100V -> (none)
- C21: value 10uF x 10V -> (none)
- C24, C9: value 1uF -> (none)
- C5: value 100nF x 50V -> (none)
- CN1: value Micro-SD Card -> MICROSD-PUSH-OUT
- CN3: value USB 3.2 Gen 2 Type C Receptacle -> USB4080-03-A
- CN4: value ARM 10-pin JTAG Connector -> FTSH-105-01-L-DV-K-TR
- DS1: value SSD1306 -> DISPLAY-OLED-128X64
- G1: value CR1220 -> CH291-1220LF
- IC2: value MCP73831/2 -> MCP73831/OT
- Q2, Q3: value SI2374DS -> SI2374DSTRPBF
- Q4: value BC817 -> BC817-16LT1SMD
- R1, R2: value 5k1 (5%) -> (none)
- R10: value 4k7 -> (none)
- R11, R15, R5: value 10k (5%) -> (none)
- R12: value 4K7 -> (none)
- R13: value 2k -> (none)
- R14: value 4K7 (5%) -> (none)
- R17: value 1k (5%) -> (none)
- R18: value 10k -> (none)
- R22: value 470R -> (none)
- R3, R41, R42: value 1M -> (none)
- R4, R9: value 100k -> (none)
- R6, R7, R8: value 47k (5%) -> (none)
- U1: value SN74AHC1G125DRLR -> SN74AHC1G125
- X2: value 32.768 kHz -> CRYSTAL-MINI
Connections:
- removed net N$17: C10.2, C11.2, R10.2, R17.1, U2.VDD, U2.VDDA
- new net N$11: C10.2, C11.2, R10.1, R17.1, U2.VDD, U2.VDDA
- net 0V: now also C10.1, C11.1, C7.1
- net N$12: now also R10.2; no longer R10.1
- net VUSB: now also C7.2
Other:
- moved on the sheet: C1, C10, C11, C14, C15, C16, C2, C21, C5, C6, C7, CN2-1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

Commit message: WIP
Parts:
- C1, C10, C11, C15, C16, C19, C24, C25, C3, C39, C4, C7, C8, C9: device rcl:C-EUC0603 -> My-RLC:C_0603
- C14: device rcl:C-EUC0805 -> My-RLC:C_0603
- CN3: value USB4080-03-A -> USB 3.2 Gen 2 Type C Receptacle
- R1, R10, R11, R12, R13, R14, R15, R17, R18, R2, R22, R3, R4, R41, R42, R5, R9: device rcl:R-EU_R0603 -> My-RLC:R_0603
