File: Hardware/0. Project/NoteIt.sch (EAGLE design)
At the start: 65 parts, among them CN1 USB 3.2 Gen 2 Type C Receptac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, CN2 Lithium Ion Polymer, CN3 OSTTE020104, CN4 FTSH-105-01-L-DV-K-TR, CN5 CR1220, CN6 Micro-SD Card, Q1 BC817, Q2 SI2374DS, Q3 SI2374DS, SW1 KY-040, U1 MCP73831/2, U2 MSP430FR2476TPTR, U3 S-8261ACMMD-G4MT2U, U4 GL823K, U5 SN74AHC1G125DBV, U6 TS3A27518EPWR, U7 TLV75530PDBVR, U8 DS3231/SO, Y1 32.768 kHz

Commit message: WIP
Parts:
- C1: value 10uF x 10V -> 10uF; PARTNO (none) -> *
- C10, C11, C12, C14, C15, C16, C17, C18, C19, C2, C20, C21, C3, C4, C5, C6, C7, CN1, CN2, CN3, CN4, CN5, CN6, DS1, LED1, Q1, Q2, Q3, R1, R11, R12, R15, R16, R2, R4, R7, R9, SW1, U1, U2, U3, U4, U5, U6, U7, U8, Y1: PARTNO (none) -> *
- C13: value 1nF x 50V -> 1nF; PARTNO (none) -> *
- C8, C9: value 22pF x 100V -> 22pF; PARTNO (none) -> *
- R10, R19, R20: value 4K7 (5%) -> 4k7; PARTNO (none) -> *
- R13, R18, R21, R22, R23, R8: value 10k (5%) -> 10k; PARTNO (none) -> *
- R14: value 1k (5%) -> 1k; PARTNO (none) -> *
- R17: value 47k (5%) -> 47k; PARTNO (none) -> *
- R3, R6: value 5k1 (5%) -> 5k1; PARTNO (none) -> *
- R5: value 4K7 -> 4k7; PARTNO (none) -> *
Connections:
- net N$33 renamed VBAT
- net 0V: no longer CN4.7
- net USB_N: now also CN1.DN2, U4.DN; no longer CN1.DP2, U4.DP
- net USB_P: now also CN1.DP2, U4.DP; no longer CN1.DN2, U4.DN
Other:
- note added: "1.3"
- note removed: "1.2"

Commit message: PCB revision WIP
Other:
- note added: "2.0"
- note removed: "1.3"

Commit message: PCB revision WIP
Other:
- note added: "I-REG = 213mA"
Changed lines of the file:
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@@
 from SIMO (MOSI) pin.</text>
 <text x="322.072" y="97.536" size="2.54" layer="200" align="center-left" grouprefs="DISPLAY_OLED">*</text>
+<text x="76.835" y="330.708" size="1.27" layer="205" font="vector" align="center">I-REG = 213mA</text>
 </plain>
 <instances>

Commit message: Schematic minor improvements and bug fix to pre PCB v3.0 release
- Fix bug at USB DP and DN.
- Change all parts to my own libraries.
Parts:
- removed CN4: FTSH-105-01-L-DV-K-TR, SamacSys_Parts:FTSH-105-01-L-DV-K-TR
- removed DS1: DISPLAY-OLED-128X64, diy-modules:DISPLAY-OLED-128X64
- added CN7: JTAG, My-Connectors:JTAG
- added CN9: OLED-MODULE-SPI-NO_HOLES, My-Displays:OLED-MODULE-SPI-NO_HOLES
- C3: PN (none) -> test
- CN1: value USB 3.2 Gen 2 Type C Receptacle -> USB Type C Receptacle; device USB C CONNECOTR:USB4080-03-A -> My-Connectors:USB-C-16P-2LAYERS; PARTNO * -> (none)
- CN2: value Lithium Ion Polymer -> CELL-JST-PH-2P-H; device Battery:BATTERYJST-2 -> My-Battery:CELL-JST-PH-2P-H; CAPACITY (none) -> 2000mAh; PARTNO * -> (none); TYPE (none) -> Li-Po; VOLTAGE (none) -> 3.7V~4.2V
- CN3: value OSTTE020104 -> 2P-BLOCK-3.5MM-2P; device Terminal Block 2P 3.5pitch:OSTTE020104 -> My-Connectors:2P-BLOCK-3.5MM-2P; PARTNO * -> (none)
- CN5: value CR1220 -> CR-1225; device SamacSys_Parts:CR1220 -> My-Battery:CR-1225
- CN6: value Micro-SD Card -> Micro SD-Card; device Micro SD:MICROSD-PUSH-OUT -> My-Sockets:SD-CARD
- LED1: value (none) -> LED-0603; device led:LEDCHIPLED_0603 -> My-LEDs:LED-0603; FAMILY (none) -> Green; PARTNO * -> (none)
- Q1: device transistor-npn:BC817-16LT1SMD -> My-Transistors:NPN-BC817
- Q2, Q3: value SI2374DS -> N-FET-ENHANCEMENT-SQ2310; device SI2374DS:SI2374DSSOT23 -> My-Transistors:N-FET-ENHANCEMENT-SQ2310
- SW1: device rotary-encoder:KY-040 -> My-Electromechanicals:ROTARY-ENCODER
- U1: device adafruit:MCP73831/OT -> My-ICs:MCP73831T-2ACI/OT
- U2: device MSP430FR2476TPTR:MSP430FR2476TPTR -> My-Microcontrollers:MSP430FR2476TPTR
- U3: value S-8261ACMMD-G4MT2U -> S-8261; device SamacSys_Parts:S-8261ACMMD-G4MT2U -> My-ICs:S-8261
- U4: device SamacSys_Parts:GL823K -> My-ICs:GL823K
- U5: value SN74AHC1G125DBV -> SN74AHC1G125; device SN74AHC1G125DRLR:SN74AHC1G125DBV -> My-ICs:SN74AHC1G125
- U6: value TS3A27518EPWR -> TS3A27518E; device TS3A27518EPWR:TS3A27518EPWR -> My-ICs:TS3A27518E
- U7: device TLV75530PDBVR:TLV75530PDBVR -> My-LDOs:TLV75530PDBVR
- U8: value DS3231/SO -> DS3231-SO16; device adafruit:DS3231/SO -> My-ICs:DS3231-SO16
- Y1: device crystal-geyer_V1_0:CRYSTAL-MINI -> My-Crystals:OSC-32.768KHZ
Connections:
- removed net N$21: CN1.CC2, R6.1
- removed net USB_N: CN1.DN1, CN1.DN2, U4.DN
- removed net USB_P: CN1.DP1, CN1.DP2, U4.DP
- new net N$17: CN1.D+, U4.DP
- new net N$18: CN1.D-, U4.DN
- new net N$19: CN1.CC1, R6.1
- net !GPIO_DISPLAY_RESET: now also CN9.!RST; no longer DS1.!RST
- net !SPI_DISPLAY_CS: now also CN9.!CS; no longer DS1.!CS
- net 0V: now also CN1.GND, CN3-2.P$1, CN7.GND, CN7.GND2, CN7.GND3, CN9.GND; no longer CN1.GND_A, CN1.GND_B, CN3.2, CN4.3, CN4.5, CN4.9, DS1.GND
- net 3.3V: now also CN7.VDD, CN9.VCC; no longer CN4.1, DS1.VCC
- net GPIO_DISPLAY_TRANSMISSION_MODE: now also CN9.DC; no longer DS1.DC
- net ICSP_SBWTCK: now also CN7.TCK; no longer CN4.4
- net ICSP_SBWTDIO: now also CN7.TDO; no longer CN4.6
- net N$10: now also CN1.S1, CN1.S2, CN1.S3, CN1.S4; no longer CN1.SHIELD
- net N$32: now also CN2.-; no longer CN2.GND
- net N$4: now also CN3-1.P$1; no longer CN3.1
- net N$5: now also LED1.K; no longer LED1.C
- net N$6: now also CN1.CC2; no longer CN1.CC1
- net SPI_DISPLAY_SCLK: now also CN9.SCLK; no longer DS1.SCLK
- net SPI_DISPLAY_SIMO: now also CN9.MOSI; no longer DS1.MOSI
- net VBAT: now also CN2.+; no longer CN2.VDD
- net VUSB: now also CN1.VBUS; no longer CN1.VBUS_A, CN1.VBUS_B
Other:
- note removed: "(3V / 37 mAh)"
- note removed: "2.0"
- note removed: "3.7V ~ 4.2V 230mAh"
- note removed: "Complete Schematic"
- note removed: "Tiago Silva"
- note removed: "github.com/TiagoPaulaSilva/NoteIt"
- moved on the sheet: C21, C3, CN6, Q2, Q3, R3, R4, R6, U1, U7

Commit message: PCB v2.0 release
Parts:
- removed CN9: OLED-MODULE-SPI-NO_HOLES, My-Displays:OLED-MODULE-SPI-NO_HOLES
- added CN4: JTAG, My-Connectors:JTAG
- CN7: value JTAG -> OLED-MODULE-SPI-NO_HOLES; device My-Connectors:JTAG -> My-Displays:OLED-MODULE-SPI-NO_HOLES; PARTNO (none) -> *
- R10: value 4k7 -> 470R
- R3: value 5k1 -> 4k7
- R5: value 4k7 -> 5k1
- R9: value 470R -> 4k7
Connections:
- net !GPIO_DISPLAY_RESET: now also CN7.!RST; no longer CN9.!RST
- net !SPI_DISPLAY_CS: now also CN7.!CS; no longer CN9.!CS
- net 0V: now also CN4.GND, CN4.GND2, CN4.GND3, R3.1, R5.2; no longer CN7.GND2, CN7.GND3, CN9.GND, R3.2, R5.1
- net 3.3V: now also CN4.VDD, CN7.VCC; no longer CN7.VDD, CN9.VCC
- net GPIO_DISPLAY_TRANSMISSION_MODE: now also CN7.DC; no longer CN9.DC
- net ICSP_SBWTCK: now also CN4.TCK; no longer CN7.TCK
- net ICSP_SBWTDIO: now also CN4.TDO; no longer CN7.TDO
- net N$14: now also R9.1; no longer R10.1
- net N$26: now also R3.2; no longer R5.2
- net N$31: now also R10.2; no longer R9.2
- net N$6: now also R5.1; no longer R3.1
- net SPI_DISPLAY_SCLK: now also CN7.SCLK; no longer CN9.SCLK
- net SPI_DISPLAY_SIMO: now also CN7.MOSI; no longer CN9.MOSI
- net VBAT: now also R10.1; no longer R9.1
- net VUSB: now also R9.2; no longer R10.2
Other:
- moved on the sheet: C7, CN2, CN3-1, CN3-2, Q2, Q3, R10, R15, R16, R3, R5, R7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

Commit message: PCB v2.0 release
Parts:
- U3: SPICEPREFIX (none) -> X
Changed lines of the file:
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@@
 <setting verticaltext="up"/>
 </settings>
-<grid distance="0.1" unitdist="inch" unit="inch" style="lines" multiple="1" display="no" altdistance="0.0125" altunitdist="inch" altunit="inch"/>
+<grid distance="0.025" unitdist="inch" unit="inch" style="lines" multiple="1" display="no" altdistance="0.0125" altunitdist="inch" altunit="inch"/>
 <layers>
 <layer number="1" name="Top" color="59" fill="1" visible="no" active="no"/>
@@
 <attribute name="PARTNO" value="*"/>
 </part>
-<part name="U3" library="My-ICs" library_urn="urn:adsk.eagle:library:35512106" deviceset="S-8261" device="" package3d_urn="urn:adsk.eagle:package:36225862/1" value="S-8261">
-<attribute name="PARTNO" value="*"/>
+<part name="U3" library="My-ICs" library_urn="urn:adsk.eagle:library:35512106" deviceset="S-8261" device="" package3d_urn="urn:adsk.eagle:package:36225862/1" override_package3d_urn="urn:adsk.eagle:package:36228518/2" override_package_urn="urn:adsk.eagle:footprint:36225858/1" value="S-8261">
+<attribute name="PARTNO" value="*"/>
+<attribute name="SPICEPREFIX" value="X"/>
 </part>
 <part name="R7" library="My-RLC" library_urn="urn:adsk.eagle:library:35509816" deviceset="R_" device="0603" package3d_urn="urn:adsk.eagle:package:35509946/1" value="2k">
@@
 <wire x1="182.88" y1="373.38" x2="181.61" y2="374.015" width="0.1524" layer="208" grouprefs="POWER_SUPPLY BATTERY_PROTECTOR"/>
 <text x="185.039" y="375.793" size="1.27" layer="208" align="center" grouprefs="POWER_SUPPLY BATTERY_PROTECTOR">7μA max.</text>
-<text x="75.565" y="334.01" size="1.27" layer="208" font="vector" align="center" grouprefs="BATTERY_CHARGING_MANAGER POWER_SUPPLY">I-REG [mA]
+<text x="75.565" y="334.01" size="1.27" layer="208" font="vector" align="center" grouprefs="POWER_SUPPLY BATTERY_CHARGING_MANAGER">I-REG [mA]
 = 1000V / R-PROG</text>
-<wire x1="104.14" y1="379.73" x2="110.49" y2="379.73" width="0.1524" layer="208" grouprefs="BATTERY_CHARGING_MANAGER POWER_SUPPLY"/>
-<wire x1="110.49" y1="379.73" x2="109.22" y2="379.095" width="0.1524" layer="208" grouprefs="BATTERY_CHARGING_MANAGER POWER_SUPPLY"/>
-<wire x1="109.22" y1="379.095" x2="109.22" y2="380.365" width="0.1524" layer="208" grouprefs="BATTERY_CHARGING_MANAGER POWER_SUPPLY"/>
-<wire x1="109.22" y1="380.365" x2="110.49" y2="379.73" width="0.1524" layer="208" grouprefs="BATTERY_CHARGING_MANAGER POWER_SUPPLY"/>
-<text x="108.331" y="376.682" size="1.27" layer="208" rot="R180" align="center" grouprefs="BATTERY_CHARGING_MANAGER POWER_SUPPLY">15mA to
+<wire x1="104.14" y1="379.73" x2="110.49" y2="379.73" width="0.1524" layer="208" grouprefs="POWER_SUPPLY BATTERY_CHARGING_MANAGER"/>
+<wire x1="110.49" y1="379.73" x2="109.22" y2="379.095" width="0.1524" layer="208" grouprefs="POWER_SUPPLY BATTERY_CHARGING_MANAGER"/>
+<wire x1="109.22" y1="379.095" x2="109.22" y2="380.365" width="0.1524" layer="208" grouprefs="POWER_SUPPLY BATTERY_CHARGING_MANAGER"/>
+<wire x1="109.22" y1="380.365" x2="110.49" y2="379.73" width="0.1524" layer="208" grouprefs="POWER_SUPPLY BATTERY_CHARGING_MANAGER"/>
+<text x="108.331" y="376.682" size="1.27" layer="208" rot="R180" align="center" grouprefs="POWER_SUPPLY BATTERY_CHARGING_MANAGER">15mA to
 500mA max.</text>
 <text x="332.105" y="393.065" size="1.778" layer="208" align="center" grouprefs="POWER_SUPPLY VOLTAGE_REGULATOR">238mV drops
@@
 <text x="259.08" y="395.605" size="0.254" layer="201" align="center" grouprefs="POWER_SUPPLY BATTERY_MONITOR"> </text>
 <text x="185.42" y="395.605" size="0.254" layer="91" align="center" grouprefs="POWER_SUPPLY BATTERY_PROTECTOR"> </text>
-<text x="44.45" y="395.605" size="0.254" layer="91" align="center" grouprefs="BATTERY_CHARGING_MANAGER POWER_SUPPLY"> </text>
+<text x="44.45" y="395.605" size="0.254" layer="91" align="center" grouprefs="POWER_SUPPLY BATTERY_CHARGING_MANAGER"> </text>
 <wire x1="249.555" y1="236.855" x2="278.765" y2="236.855" width="0.254" layer="204" style="shortdash" grouprefs="MICRO_SDCARD_CONTROLLER"/>
 <wire x1="278.765" y1="236.855" x2="278.765" y2="213.995" width="0.254" layer="204" style="shortdash" grouprefs="MICRO_SDCARD_CONTROLLER"/>
@@
 <attribute name="VALUE" x="458.47" y="188.341" size="1.27" layer="96"/>
 </instance>
-<instance part="U1" gate="G$1" x="90.17" y="368.935" smashed="yes" grouprefs="BATTERY_CHARGING_MANAGER POWER_SUPPLY">
+<instance part="U1" gate="G$1" x="90.17" y="368.935" smashed="yes" grouprefs="POWER_SUPPLY BATTERY_CHARGING_MANAGER">
 <attribute name="PARTNO" x="90.17" y="368.935" size="1.778" layer="96" display="off"/>
 <attribute name="NAME" x="77.47" y="387.985" size="1.778" layer="95"/>
 <attribute name="VALUE" x="77.47" y="385.445" size="1.778" layer="96"/>
 </instance>
-<instance part="R3" gate="G$1" x="62.23" y="334.01" smashed="yes" rot="R90" grouprefs="BATTERY_CHARGING_MANAGER POWER_SUPPLY">
+<instance part="R3" gate="G$1" x="62.23" y="334.01" smashed="yes" rot="R90" grouprefs="POWER_SUPPLY BATTERY_CHARGING_MANAGER">
 <attribute name="NAME" x="60.0964" y="334.01" size="1.27" layer="95" rot="R90" align="center"/>
 <attribute name="VALUE" x="64.262" y="334.01" size="1.27" layer="96" rot="R90" align="center"/>
@@
 <segment>
 <pinref part="R3" gate="G$1" pin="1"/>
-<wire x1="62.23" y1="328.93" x2="62.23" y2="313.69" width="0.1524" layer="91" grouprefs="BATTERY_CHARGING_MANAGER POWER_SUPPLY"/>
+<wire x1="62.23" y1="328.93" x2="62.23" y2="313.69" width="0.1524" layer="91" grouprefs="POWER_SUPPLY BATTERY_CHARGING_MANAGER"/>
 <pinref part="U1" gate="G$1" pin="VSS"/>
-<wire x1="88.9" y1="342.265" x2="88.9" y2="313.69" width="0.1524" layer="91" grouprefs="BATTERY_CHARGING_MANAGER POWER_SUPPLY"/>
-<wire x1="88.9" y1="313.69" x2="62.23" y2="313.69" width="0.1524" layer="91" grouprefs="BATTERY_CHARGING_MANAGER POWER_SUPPLY"/>
+<wire x1="88.9" y1="342.265" x2="88.9" y2="313.69" width="0.1524" layer="91" grouprefs="POWER_SUPPLY BATTERY_CHARGING_MANAGER"/>
+<wire x1="88.9" y1="313.69" x2="62.23" y2="313.69" width="0.1524" layer="91" grouprefs="POWER_SUPPLY BATTERY_CHARGING_MANAGER"/>
 <pinref part="R7" gate="G$1" pin="1"/>
 <wire x1="125.73" y1="313.69" x2="125.73" y2="316.23" width="0.1524" layer="91" grouprefs="POWER_SUPPLY"/>
 <junction x="125.73" y="313.69" grouprefs="POWER_SUPPLY"/>
 <wire x1="88.9" y1="313.69" x2="125.73" y2="313.69" width="0.1524" layer="91" grouprefs="POWER_SUPPLY"/>
-<junction x="88.9" y="313.69" grouprefs="BATTERY_CHARGING_MANAGER POWER_SUPPLY"/>
+<junction x="88.9" y="313.69" grouprefs="POWER_SUPPLY BATTERY_CHARGING_MANAGER"/>
 <wire x1="217.805" y1="326.39" x2="217.805" y2="313.69" width="0.1524" layer="91" grouprefs="POWER_SUPPLY"/>
 <wire x1="217.805" y1="313.69" x2="125.73" y2="313.69" width="0.1524" layer="91" grouprefs="POWER_SUPPLY"/>
@@
 <pinref part="U1" gate="G$1" pin="PROG"/>
 <pinref part="R3" gate="G$1" pin="2"/>
-<wire x1="72.39" y1="353.695" x2="62.23" y2="353.695" width="0.1524" layer="91" grouprefs="BATTERY_CHARGING_MANAGER POWER_SUPPLY"/>
-<wire x1="62.23" y1="353.695" x2="62.23" y2="339.09" width="0.1524" layer="91" grouprefs="BATTERY_CHARGING_MANAGER POWER_SUPPLY"/>
+<wire x1="72.39" y1="353.695" x2="62.23" y2="353.695" width="0.1524" layer="91" grouprefs="POWER_SUPPLY BATTERY_CHARGING_MANAGER"/>
+<wire x1="62.23" y1="353.695" x2="62.23" y2="339.09" width="0.1524" layer="91" grouprefs="POWER_SUPPLY BATTERY_CHARGING_MANAGER"/>
 </segment>
 </net>
